Commit message: Added controllers for movemnt

File: amr_with_arm_description/urdf/amr_with_arm.xacro (robot description, xacro)
@@ -1,4 +1,4 @@
 <?xml version="1.0"?>
-<robot xmlns:xacro="http://ros.org/wiki/xacro" name="amr_with_arm">
+<robot name="amr_with_arm" xmlns:xacro="http://www.ros.org/wiki/xacro">
   <!-- Load mobile robot -->
   <xacro:include filename="$(find bot_description)/urdf/bot.xacro"/>
@@ -7,7 +7,49 @@
   <!-- Fixed joint to attach arm to AMR -->
   <joint name="arm_mount" type="fixed">
-    <parent link="base_footprint"/> <!-- Replace with your AMR's base link -->
-    <child link="$(arg prefix)link1"/> <!-- Replace with arm's base link -->
-    <origin xyz="0 0 0.4" rpy="0 0 0"/> <!-- Adjust height and position -->
+    <parent link="base_footprint"/>
+    <child link="$(arg prefix)link1"/>
+    <origin xyz="0 0 0.4" rpy="0 0 0"/>
   </joint>
+  <!-- ros2_control for AMR base (diff drive) -->
+  <ros2_control name="amr_base_system" type="system">
+    <hardware>
+      <plugin>gazebo_ros2_control/GazeboSystem</plugin>
+    </hardware>
+    <joint name="left_wheel_joint">
+      <command_interface name="velocity"/>
+      <state_interface name="position"/>
+      <state_interface name="velocity"/>
+    </joint>
+    <joint name="right_wheel_joint">
+      <command_interface name="velocity"/>
+      <state_interface name="position"/>
+      <state_interface name="velocity"/>
+    </joint>
+  </ros2_control>
+  <!-- ros2_control for arm -->
+  <ros2_control name="amr_with_arm_arm_system" type="system">
+    <hardware>
+      <plugin>gazebo_ros2_control/GazeboSystem</plugin>
+    </hardware>
+    <joint name="joint1">
+      <command_interface name="position"/>
+      <state_interface name="position"/>
+      <state_interface name="velocity"/>
+    </joint>
+    <joint name="joint2">
+      <command_interface name="position"/>
+      <state_interface name="position"/>
+      <state_interface name="velocity"/>
+    </joint>
+    <joint name="joint3">
+      <command_interface name="position"/>
+      <state_interface name="position"/>
+      <state_interface name="velocity"/>
+    </joint>
+    <joint name="joint4">
+      <command_interface name="position"/>
+      <state_interface name="position"/>
+      <state_interface name="velocity"/>
+    </joint>
+  </ros2_control>
 </robot>

File: bot/bot_description/urdf/bot.xacro (robot description, xacro)
@@ -98,5 +98,5 @@
   </collision>
 </link>
-<joint name="Revolute1" type="continuous">
+<joint name="right_wheel_joint" type="continuous">
   <origin xyz="0.0 -0.2 0.05" rpy="0 0 0"/>
   <parent link="base_link"/>
@@ -109,5 +109,5 @@
   <child link="lidar_1"/>
 </joint>
-<joint name="Revolute3" type="continuous">
+<joint name="left_wheel_joint" type="continuous">
   <origin xyz="0.0 0.2 0.05" rpy="0 0 0"/>
   <parent link="base_link"/>

File: open_manipulator_x/open_manipulator_x_description/ros2_control/open_manipulator_x_system.ros2_control.xacro (robot description, xacro)
@@ -8,5 +8,5 @@
         </hardware>
       </xacro:if>
-      <xacro:unless value="$(arg use_sim)">
+      <!-- <xacro:unless value="$(arg use_sim)">
         <hardware>
           <xacro:if value="${use_fake_hardware}">
@@ -44,6 +44,4 @@
             <param name="reboot_dxl_srv_name">dynamixel_hardware_interface/reboot_dxl</param>
             <param name="set_dxl_torque_srv_name">dynamixel_hardware_interface/set_dxl_torque</param>
-              <!-- This parameter is used for a prismatic joint
-            that operates through a revolute mechanism. If the joint does not require this configuration, this parameter can be removed. -->
             <param name="use_revolute_to_prismatic_gripper">1</param>
             <param name="revolute_to_prismatic_dxl">dxl5</param>
@@ -55,5 +53,5 @@
           </xacro:unless>
         </hardware>
-      </xacro:unless>
+      </xacro:unless> -->
       <joint name="${prefix}joint1">
         <command_interface name="position"/>
@@ -94,5 +92,5 @@
         <state_interface name="effort"/>
       </joint>
-      <gpio name="dxl1">
+      <!-- <gpio name="dxl1">
         <param name="type">dxl</param>
         <param name="ID">11</param>
@@ -172,5 +170,5 @@
         <state_interface name="Present Input Voltage"/>
         <param name="Return Delay Time">0</param>
-      </gpio>
+      </gpio> -->
     </ros2_control>
   </xacro:macro>

Commit message: chnage teh arm position

File: amr_with_arm_description/urdf/amr_with_arm.xacro (robot description, xacro)
@@ -9,5 +9,5 @@
     <parent link="base_footprint"/>
     <child link="$(arg prefix)link1"/>
-    <origin xyz="0 0 0.4" rpy="0 0 0"/>
+    <origin xyz="-0.1 0 0.03" rpy="0 0 3.1416"/>
   </joint>
   <!-- ros2_control for AMR base (diff drive) -->

Commit message: Changed  teh world , error correction

File: amr_with_arm_description/urdf/amr_with_arm.xacro (robot description, xacro)
@@ -9,5 +9,5 @@
     <parent link="base_footprint"/>
     <child link="$(arg prefix)link1"/>
-    <origin xyz="-0.1 0 0.03" rpy="0 0 3.1416"/>
+    <origin xyz="-0.1 0 0.08" rpy="0 0 3.1416"/>
   </joint>
   <!-- ros2_control for AMR base (diff drive) -->

File: bot/bot_description/urdf/bot.xacro (robot description, xacro)
@@ -31,4 +31,8 @@
     <material name="silver"/>
   </visual>
+  <inertial>
+    <mass value="0.5"/>
+    <inertia ixx="0.001" ixy="0.0" ixz="0.0" iyy="0.001" iyz="0.0" izz="0.001"/>
+  </inertial>
   <collision>
     <origin xyz="0 0 0" rpy="0 0 0"/>
@@ -57,4 +61,8 @@
     </geometry>
   </collision>
+  <inertial>
+    <mass value="0.5"/>
+    <inertia ixx="0.001" ixy="0.0" ixz="0.0" iyy="0.001" iyz="0.0" izz="0.001"/>
+  </inertial>
 </link>
 <link name="lidar_1">

Commit message: Added linear guide and its controller

File: amr_with_arm_description/urdf/amr_with_arm.xacro (robot description, xacro)
@@ -3,13 +3,15 @@
   <!-- Load mobile robot -->
   <xacro:include filename="$(find bot_description)/urdf/bot.xacro"/>
+  <!-- Load linear guide -->
+  <xacro:include filename="$(find amr_with_arm_description)/urdf/linear_guide.xacro"/>
   <!-- Load manipulator -->
   <xacro:include filename="$(find open_manipulator_x_description)/urdf/open_manipulator_x_robot.urdf.xacro"/>
-  <!-- Fixed joint to attach arm to AMR -->
+  <!-- Attach arm to linear guide moving base -->
   <joint name="arm_mount" type="fixed">
-    <parent link="base_footprint"/>
+    <parent link="linear_guide_base"/>
     <child link="$(arg prefix)link1"/>
     <origin xyz="-0.1 0 0.08" rpy="0 0 3.1416"/>
   </joint>
-  <!-- ros2_control for AMR base (diff drive) -->
+  <!-- ROS2 Control for mobile robot (diff drive) -->
   <ros2_control name="amr_base_system" type="system">
     <hardware>
@@ -27,9 +29,16 @@
     </joint>
   </ros2_control>
-  <!-- ros2_control for arm -->
+  <!-- ROS2 Control for arm and linear guide -->
   <ros2_control name="amr_with_arm_arm_system" type="system">
     <hardware>
       <plugin>gazebo_ros2_control/GazeboSystem</plugin>
     </hardware>
+    <!-- Linear guide prismatic joint -->
+    <joint name="linear_guide_prismatic_joint">
+      <command_interface name="position"/>
+      <state_interface name="position"/>
+      <state_interface name="velocity"/>
+    </joint>
+    <!-- OpenManipulator X joints -->
     <joint name="joint1">
       <command_interface name="position"/>
